File: Hardware/14140.brd (EAGLE design)
At the start: 78.7 x 66 mm, 157 parts, among them J1 PST1,0/4-3,5, J10 PPPC101LFBN, J11 ICSP, J2 PST1,0&8-3,5, J3 PST1,0/3-3,5, J4 PST1,0/5-3,5, J5 PPPC101LFBN, J6 PPPC081LFBN, J7 PST1,0/6-3,5, J9 PPPC101LFBN, Q1 DMB, Q10 K84, Q11 K3N, Q12 K3N, Q13 K38, Q14 K3N, Q15 K3N, Q16 K3N, Q17 K3N, Q18 DMB, Q19 K38, Q2 K38, Q20 K1N, Q21 K38, Q22 K1N, Q23 K38, Q24 K1N, Q25 K38, Q26 K1N, Q27 K1N, Q28 K38, Q29 K1N, Q3 K1N, Q30 K38, Q31 K38, Q32 K1N, Q33 K3N, Q34 K3N, Q4 K1N, Q5 DMB, Q6 34N, Q7 K3N, Q8 K3N, Q9 K38, U1 LT3652, U2 I50115, U3 1087, U4 1087, U5 TPS3700, U6 ATMEGA328PB-AU, Y1 16MHz

Commit message: Adc: ch7 can now read PWR (e.g. battery)
up to 15V (was 7.5V for 6V SLA)
Parts:
- R36: value 100k -> 200k
- R37: value 200k -> 100k
Changed lines of the file:
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@@
 <attribute name="VALUE" x="8.001" y="9.271" size="0.4064" layer="27" rot="R180"/>
 </element>
-<element name="R36" library="R-C" package="C0805(2012)" value="100k" x="34.417" y="52.07" smashed="yes" rot="R180">
+<element name="R36" library="R-C" package="C0805(2012)" value="200k" x="34.417" y="52.07" smashed="yes" rot="R180">
 <attribute name="NAME" x="32.004" y="52.705" size="0.6096" layer="25" rot="R270"/>
 <attribute name="VALUE" x="35.306" y="52.324" size="0.4064" layer="27" rot="R180"/>
 </element>
-<element name="R37" library="R-C" package="C0805(2012)" value="200k" x="33.274" y="54.102" smashed="yes">
+<element name="R37" library="R-C" package="C0805(2012)" value="100k" x="33.274" y="54.102" smashed="yes">
 <attribute name="NAME" x="34.036" y="55.753" size="0.6096" layer="25" rot="R180"/>
 <attribute name="VALUE" x="32.385" y="53.848" size="0.4064" layer="27"/>
