File: Hardware/14140.sch (EAGLE design)
At the start: 157 parts, among them J1 PST1,0/4-3,5, J10 PPPC101LFBN, J11 ICSP, J2 PST1,0&8-3,5, J3 PST1,0/3-3,5, J4 PST1,0/5-3,5, J5 PPPC101LFBN, J6 PPPC081LFBN, J7 PST1,0/6-3,5, J9 PPPC101LFBN, Q1 DMB, Q10 K84, Q11 K3N, Q12 K3N, Q13 K38, Q14 K3N, Q15 K3N, Q16 K3N, Q17 K3N, Q18 DMB, Q19 K38, Q2 K38, Q20 K1N, Q21 K38, Q22 K1N, Q23 K38, Q24 K1N, Q25 K38, Q26 K1N, Q27 K1N, Q28 K38, Q29 K1N, Q3 K1N, Q30 K38, Q31 K38, Q32 K1N, Q33 K3N, Q34 K3N, Q4 K1N, Q5 DMB, Q6 34N, Q7 K3N, Q8 K3N, Q9 K38, U1 LT3652, U2 I50115, U3 1087, U4 1087, U5 TPS3700, U6 ATMEGA328PB-AU, Y1 16MHz

Commit message: Adc: ch7 can now read PWR (e.g. battery)
up to 15V (was 7.5V for 6V SLA)
Parts:
- R36: value 100k -> 200k
- R37: value 200k -> 100k
Other:
- note added: "PWR * .333"
- note removed: "PWR * .667"
Changed lines of the file:
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@@
 <part name="GND22" library="Plane" deviceset="0V" device=""/>
 <part name="R34" library="R-C" deviceset="R" device="0805" value="432k"/>
-<part name="R36" library="R-C" deviceset="R" device="0805" value="100k"/>
-<part name="R37" library="R-C" deviceset="R" device="0805" value="200k"/>
+<part name="R36" library="R-C" deviceset="R" device="0805" value="200k"/>
+<part name="R37" library="R-C" deviceset="R" device="0805" value="100k"/>
 <part name="C19" library="C-C" deviceset="C" device="C0603A" value=".01uF"/>
 <part name="GND42" library="Plane" deviceset="0V" device=""/>
@@
 <text x="171.196" y="126.492" size="2.54" layer="98">PV AND BATTERY VOLTAGE</text>
 <text x="146.304" y="123.19" size="1.27" layer="98">PV * .188</text>
-<text x="204.724" y="123.19" size="1.27" layer="98">PWR * .667</text>
+<text x="204.724" y="123.19" size="1.27" layer="98">PWR * .333</text>
 <text x="7.62" y="24.13" size="1.778" layer="98">ECS-160-20-3X-TR
 16MHZ +/- 30PPM
