File: Hardware/Design/14140.brd (EAGLE design)
At the start: 78.7 x 66 mm, 157 parts, among them J1 PST1,0/4-3,5, J10 PPPC101LFBN, J11 ICSP, J2 PST1,0&8-3,5, J3 PST1,0/3-3,5, J4 PST1,0/5-3,5, J5 PPPC101LFBN, J6 PPPC081LFBN, J7 PST1,0/6-3,5, J9 PPPC101LFBN, Q1 DMB, Q10 K84, Q11 K3N, Q12 K3N, Q13 K38, Q14 K3N, Q15 K3N, Q16 K3N, Q17 K3N, Q18 DMB, Q19 K38, Q2 K38, Q20 K1N, Q21 K38, Q22 K1N, Q23 K38, Q24 K1N, Q25 K38, Q26 K1N, Q27 K1N, Q28 K38, Q29 K1N, Q3 K1N, Q30 K38, Q31 K38, Q32 K1N, Q33 K3N, Q34 K3N, Q4 K1N, Q5 DMB, Q6 34N, Q7 K3N, Q8 K3N, Q9 K38, U1 LT3652, U2 I50115, U3 1087, U4 1087, U5 TPS3700, U6 ATMEGA328PB-AU, Y1 16MHz

Commit message: Hardware: ^6 review
Parts:
- moved R38 0.13 mm to (75.3, 14.0)
Connections:
- removed net N$12: Q10.3(D), Q15.E, Q17.E, R39.2, R41.2
- removed net N$5: D1.A, J1.4
- new net CS_PWR: Q10.3(D), Q12.E, Q15.E, Q17.E, Q34.E, Q8.E, R16.2, R29.2, R39.2, R41.2, R58.2
- new net PV_RAW: D1.A, J1.4, R34.2
- net PV_IN: no longer R34.2
- net VIN: no longer Q12.E, Q34.E, Q8.E, R16.2, R29.2, R58.2
Routing:
- net CS_PWR: track 0.00 -> 61.8 mm, vias 0 -> 5
- net N$12: track 24.4 -> 0.00 mm, vias 2 -> 0
- net VIN: track 166.4 -> 154.1 mm, vias 13 -> 10
- net PV_RAW: track 0.00 -> 9.67 mm
- net N$5: track 5.99 -> 0.00 mm
- net N$20: track 7.80 -> 10.9 mm, vias 2 -> 0
- net N$29: track 10.1 -> 11.5 mm
- net PV_IN: track 44.5 -> 45.2 mm, vias 1 -> 3
- net N$123: vias 0 -> 2
Other:
- board text added: "14140^6"
- board text added: "RPUBUS.ORG"
- board text removed: "14140^5"
- board text removed: "EPCCS.ORG"

Commit message: SelfTest: not done yet but a good save point
Connections:
- net SHLD_VIN renamed VOUT
Changed lines of the file:
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@@
 <wire x1="52.666" y1="59.094" x2="52.07" y2="59.69" width="0.254" layer="1"/>
 </signal>
-<signal name="SHLD_VIN">
+<signal name="VOUT">
 <contactref element="J6" pad="1"/>
 <contactref element="Q18" pad="3(D)"/>

Commit message: Hardware: circuit node names for bat-discon and vin-discon
Connections:
- net 5V88PL-DWN renamed BAT-DISCON
- net 6V58PL-DWN renamed VIN-DISCON
Changed lines of the file:
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@@
 <wire x1="14.185" y1="23.583" x2="14.224" y2="23.622" width="0.254" layer="1"/>
 </signal>
-<signal name="5V88PL-DWN">
+<signal name="BAT-DISCON">
 <contactref element="R14" pad="2"/>
 <contactref element="D3" pad="C"/>
@@
 <wire x1="36.703" y1="40.894" x2="37.167" y2="41.358" width="0.254" layer="1"/>
 </signal>
-<signal name="6V58PL-DWN">
+<signal name="VIN-DISCON">
 <contactref element="Q2" pad="3(D)"/>
 <contactref element="R4" pad="2"/>
