File: NightLight/Setup/NightLightWiring.sch (EAGLE design)
At the start: 21 parts

Commit message: NightLight: add alternate power input for solar panel
bug noted in readme
Parts:
- added PV4: PV, Documentation:PV
- added U$7: BAT, Documentation:BAT
Connections:
- removed net 12V_SLA: BM3.PWR
- removed net SLP005-12U: BM3.ALT
- new net N$1: U$7.+BAT
- new net N$42: PV4.-PV, U$7.-BAT
- new net N$50: PV4.+PV
Other:
- note added: "18AHr"
- note added: "SLP003-12U OR 17Vmp@180mA"
Changed lines of the file:
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@@
 <part name="D19" library="D-LED" deviceset="LED" device="5MM" value="RD"/>
 <part name="R1" library="R-C" deviceset="R" device="0805" value="100k"/>
+<part name="PV4" library="Documentation" deviceset="PV" device=""/>
+<part name="U$7" library="Documentation" deviceset="BAT" device=""/>
 </parts>
 <sheets>
 <sheet>
 <plain>
-<text x="28.956" y="134.366" size="5.08" layer="98">NIGHT LIGHTS</text>
+<text x="34.036" y="134.366" size="5.08" layer="98">NIGHT
+LIGHTS</text>
+<text x="87.884" y="106.172" size="2.54" layer="98" rot="R90">18AHr</text>
+<text x="91.186" y="122.936" size="2.54" layer="98" rot="R90">SLP003-12U OR
+17Vmp@180mA</text>
 </plain>
 <instances>
@@
 <instance part="D19" gate="G$1" x="20.32" y="142.24" rot="R270"/>
 <instance part="R1" gate="G$1" x="20.32" y="134.62" rot="R180"/>
+<instance part="PV4" gate="G$1" x="76.2" y="134.62"/>
+<instance part="U$7" gate="G$1" x="81.28" y="109.22" rot="R90"/>
 </instances>
 <busses>
 </busses>
 <nets>
-<net name="SLP005-12U" class="0">
-<segment>
-<label x="71.12" y="116.84" size="1.778" layer="91" xref="yes"/>
-<pinref part="BM3" gate="G$1" pin="ALT"/>
-<wire x1="71.12" y1="116.84" x2="66.04" y2="116.84" width="0.1524" layer="91"/>
-</segment>
-</net>
-<net name="12V_SLA" class="0">
-<segment>
-<label x="71.12" y="121.92" size="1.778" layer="91" xref="yes"/>
-<pinref part="BM3" gate="G$1" pin="PWR"/>
-<wire x1="71.12" y1="121.92" x2="66.04" y2="121.92" width="0.1524" layer="91"/>
-</segment>
-</net>
 <net name="DAYNIGHT_STATUS_LED" class="0">
 <segment>
@@
 </segment>
 </net>
+<net name="N$1" class="0">
+<segment>
+<pinref part="U$7" gate="G$1" pin="+BAT"/>
+<wire x1="78.74" y1="116.84" x2="78.74" y2="121.92" width="0.1524" layer="91"/>
+<wire x1="78.74" y1="121.92" x2="66.04" y2="121.92" width="0.1524" layer="91"/>
+</segment>
+</net>
+<net name="N$42" class="0">
+<segment>
+<pinref part="PV4" gate="G$1" pin="-PV"/>
+<pinref part="U$7" gate="G$1" pin="-BAT"/>
+<wire x1="73.66" y1="132.08" x2="73.66" y2="124.46" width="0.1524" layer="91"/>
+<wire x1="73.66" y1="124.46" x2="81.28" y2="124.46" width="0.1524" layer="91"/>
+<wire x1="81.28" y1="124.46" x2="81.28" y2="119.38" width="0.1524" layer="91"/>
+<wire x1="81.28" y1="119.38" x2="81.28" y2="116.84" width="0.1524" layer="91"/>
+<wire x1="66.04" y1="119.38" x2="81.28" y2="119.38" width="0.1524" layer="91"/>
+<junction x="81.28" y="119.38"/>
+</segment>
+</net>
+<net name="N$50" class="0">
+<segment>
+<pinref part="PV4" gate="G$1" pin="+PV"/>
+<wire x1="71.12" y1="116.84" x2="71.12" y2="134.62" width="0.1524" layer="91"/>
+<wire x1="71.12" y1="134.62" x2="73.66" y2="134.62" width="0.1524" layer="91"/>
+<wire x1="71.12" y1="116.84" x2="66.04" y2="116.84" width="0.1524" layer="91"/>
+</segment>
+</net>
